Commit message: #Feature lyenbot

File: src/holosoma/holosoma/data/robots/lyenbot/lyenbot_20151206.urdf (robot description, URDF)
Before this commit: robot lyenbot, 24 links, 23 joints
Links:
- link base_link: geometry collision mesh filename=meshes/base_link.STL; visual mesh filename=meshes/base_link.STL
- link left_ankle_pitch_link: geometry collision mesh filename=meshes/left_ankle_pitch_link.STL; visual mesh filename=meshes/left_ankle_pitch_link.STL
- link left_ankle_roll_link: geometry collision mesh filename=meshes/left_ankle_roll_link.STL; visual mesh filename=meshes/left_ankle_roll_link.STL
- link left_elbow_pitch_link: geometry collision mesh filename=meshes/left_elbow_pitch_link.STL; visual mesh filename=meshes/left_elbow_pitch_link.STL
- link left_elbow_roll_link: geometry collision mesh filename=meshes/left_elbow_roll_link.STL; visual mesh filename=meshes/left_elbow_roll_link.STL
- link left_elbow_yaw_link: geometry collision mesh filename=meshes/left_elbow_yaw_link.STL; visual mesh filename=meshes/left_elbow_yaw_link.STL
- link left_hip_pitch_link: geometry collision mesh filename=meshes/left_hip_pitch_link.STL; visual mesh filename=meshes/left_hip_pitch_link.STL
- link left_hip_roll_link: geometry collision mesh filename=meshes/left_hip_roll_link.STL; visual mesh filename=meshes/left_hip_roll_link.STL
- link left_hip_yaw_link: geometry collision mesh filename=meshes/left_hip_yaw_link.STL; visual mesh filename=meshes/left_hip_yaw_link.STL
- link left_knee_pitch_link: geometry collision mesh filename=meshes/left_knee_pitch_link.STL; visual mesh filename=meshes/left_knee_pitch_link.STL
- link left_shoulder_pitch_link: geometry collision mesh filename=meshes/left_shoulder_pitch_link.STL; visual mesh filename=meshes/left_shoulder_pitch_link.STL
- link left_shoulder_roll_link: geometry collision mesh filename=meshes/left_shoulder_roll_link.STL; visual mesh filename=meshes/left_shoulder_roll_link.STL
- link right_ankle_pitch_link: geometry collision mesh filename=meshes/right_ankle_pitch_link.STL; visual mesh filename=meshes/right_ankle_pitch_link.STL
- link right_ankle_roll_link: geometry collision mesh filename=meshes/right_ankle_roll_link.STL; visual mesh filename=meshes/right_ankle_roll_link.STL
- link right_elbow_pitch_link: geometry collision mesh filename=meshes/right_elbow_pitch_link.STL; visual mesh filename=meshes/right_elbow_pitch_link.STL
- link right_elbow_roll_link: geometry collision mesh filename=meshes/right_elbow_roll_link.STL; visual mesh filename=meshes/right_elbow_roll_link.STL
- link right_elbow_yaw_link: geometry collision mesh filename=meshes/right_elbow_yaw_link.STL; visual mesh filename=meshes/right_elbow_yaw_link.STL
- link right_hip_pitch_link: geometry collision mesh filename=meshes/right_hip_pitch_link.STL; visual mesh filename=meshes/right_hip_pitch_link.STL
- link right_hip_roll_link: geometry collision mesh filename=meshes/right_hip_roll_link.STL; visual mesh filename=meshes/right_hip_roll_link.STL
- link right_hip_yaw_link: geometry collision mesh filename=meshes/right_hip_yaw_link.STL; visual mesh filename=meshes/right_hip_yaw_link.STL
- link right_knee_pitch_link: geometry collision mesh filename=meshes/right_knee_pitch_link.STL; visual mesh filename=meshes/right_knee_pitch_link.STL
- link right_shoulder_pitch_link: geometry collision mesh filename=meshes/right_shoulder_pitch_link.STL; visual mesh filename=meshes/right_shoulder_pitch_link.STL
- link right_shoulder_roll_link: geometry collision mesh filename=meshes/right_shoulder_roll_link.STL; visual mesh filename=meshes/right_shoulder_roll_link.STL
- link torso: geometry collision mesh filename=meshes/torso_simple.STL; visual mesh filename=meshes/torso_simple.STL

File: src/holosoma/holosoma/data/robots/lyenbot/lyenbot_20151206_collision.urdf (robot description, URDF)
Before this commit: robot lyenbot, 24 links, 23 joints
Links:
- added link left_foot_contact_point, mass 0.001
- added link right_foot_contact_point, mass 0.001
- link base_link: geometry collision sphere radius=0.07; visual mesh filename=meshes/base_link.STL
- link left_ankle_pitch_link: geometry visual mesh filename=meshes/left_ankle_pitch_link.STL
- link left_ankle_roll_link: geometry collision cylinder length=0.05 radius=0.01; collision cylinder length=0.05 radius=0.01
- link left_elbow_pitch_link: geometry collision cylinder length=0.21 radius=0.035; visual mesh filename=meshes/left_elbow_pitch_link.STL
- link left_elbow_roll_link: geometry collision cylinder length=0.025 radius=0.045; visual mesh filename=meshes/left_elbow_roll_link.STL
- link left_elbow_yaw_link: geometry collision cylinder length=0.19 radius=0.035; visual mesh filename=meshes/left_elbow_yaw_link.STL
- link left_hip_pitch_link: geometry visual mesh filename=meshes/left_hip_pitch_link.STL
- link left_hip_roll_link: geometry collision cylinder length=0.26 radius=0.05; visual mesh filename=meshes/left_hip_roll_link.STL
- link left_hip_yaw_link: geometry visual mesh filename=meshes/left_hip_yaw_link.STL
- link left_knee_pitch_link: geometry collision cylinder length=0.26 radius=0.05; visual mesh filename=meshes/left_knee_pitch_link.STL
- link left_shoulder_pitch_link: geometry visual mesh filename=meshes/left_shoulder_pitch_link.STL
- link left_shoulder_roll_link: geometry visual mesh filename=meshes/left_shoulder_roll_link.STL
- link right_ankle_pitch_link: geometry visual mesh filename=meshes/right_ankle_pitch_link.STL
- link right_ankle_roll_link: geometry collision cylinder length=0.05 radius=0.01; collision cylinder length=0.05 radius=0.01
- link right_elbow_pitch_link: geometry collision cylinder length=0.21 radius=0.035; visual mesh filename=meshes/right_elbow_pitch_link.STL
- link right_elbow_roll_link: geometry collision cylinder length=0.025 radius=0.045; visual mesh filename=meshes/right_elbow_roll_link.STL
- link right_elbow_yaw_link: geometry collision cylinder length=0.19 radius=0.035; visual mesh filename=meshes/right_elbow_yaw_link.STL
- link right_hip_pitch_link: geometry visual mesh filename=meshes/right_hip_pitch_link.STL
- link right_hip_roll_link: geometry collision cylinder length=0.26 radius=0.05; visual mesh filename=meshes/right_hip_roll_link.STL
- link right_hip_yaw_link: geometry visual mesh filename=meshes/right_hip_yaw_link.STL
- link right_knee_pitch_link: geometry collision cylinder length=0.26 radius=0.05; visual mesh filename=meshes/right_knee_pitch_link.STL
- link right_shoulder_pitch_link: geometry visual mesh filename=meshes/right_shoulder_pitch_link.STL
- link right_shoulder_roll_link: geometry visual mesh filename=meshes/right_shoulder_roll_link.STL
- link torso: geometry collision cylinder length=0.01 radius=0.068; collision cylinder length=0.04 radius=0.056
Joints:
- added joint left_foot_contact_point: type fixed, parent left_ankle_roll_link, child left_foot_contact_point, origin xyz=0 0 -0.033 rpy=0 0 0
- added joint right_foot_contact_point: type fixed, parent right_ankle_roll_link, child right_foot_contact_point, origin xyz=0 0 -0.033 rpy=0 0 0
