Commit message: #lyenbotlegloc_fastsac_v2

File: src/holosoma/holosoma/data/robots/lyenbot/lyenbot_20260212_collision_ankle_roll_pitch.urdf (robot description, URDF)
Before this commit: robot lyenbot, 26 links, 25 joints
Joints:
- joint left_ankle_pitch_joint: limit lower=-0.611 upper=0.611 effort=66 velocity=16.22 -> lower=-0.534 upper=0.534 effort=66 velocity=16.22
- joint left_ankle_roll_joint: limit lower=-0.314 upper=0.314 effort=33 velocity=16.22 -> lower=-0.1326 upper=0.1326 effort=33 velocity=16.22
- joint right_ankle_pitch_joint: limit lower=-0.611 upper=0.611 effort=66 velocity=16.22 -> lower=-0.534 upper=0.534 effort=66 velocity=16.22
- joint right_ankle_roll_joint: limit lower=-0.314 upper=0.314 effort=33 velocity=16.22 -> lower=-0.1326 upper=0.1326 effort=33 velocity=16.22

File: src/holosoma/holosoma/data/robots/lyenbot/lyenbotlegs_20260212_collision_ankle_roll_pitch.urdf (robot description, URDF)
Before this commit: robot lyenbot, 16 links, 15 joints
Joints:
- joint left_ankle_pitch_joint: limit lower=-0.611 upper=0.611 effort=66 velocity=16.22 -> lower=-0.534 upper=0.534 effort=66 velocity=16.22
- joint left_ankle_roll_joint: limit lower=-0.314 upper=0.314 effort=33 velocity=16.22 -> lower=-0.1326 upper=0.1326 effort=33 velocity=16.22
- joint right_ankle_pitch_joint: limit lower=-0.611 upper=0.611 effort=66 velocity=16.22 -> lower=-0.534 upper=0.534 effort=66 velocity=16.22
- joint right_ankle_roll_joint: limit lower=-0.314 upper=0.314 effort=33 velocity=16.22 -> lower=-0.1326 upper=0.1326 effort=33 velocity=16.22
