Commit message: knee dof limits with 0.08

File: src/holosoma/holosoma/data/robots/lyenbot/lyenbotlegs_20260212_collision_ankle_roll_pitch.urdf (robot description, URDF)
Before this commit: robot lyenbot, 16 links, 15 joints
Joints:
- joint left_knee_pitch_joint: limit lower=0 upper=2.477 effort=140 velocity=12.04 -> lower=0.087267 upper=2.477 effort=140 velocity=12.04
- joint right_knee_pitch_joint: limit lower=0 upper=2.477 effort=140 velocity=12.04 -> lower=0.087267 upper=2.477 effort=140 velocity=12.04
